File: counter_mega/counter_mega.kicad_pcb (KiCad board)
At the start: 2 copper layers, 140.6 x 95.6 mm, 38 parts, among them J1 Screw_Terminal_01x02, J2 Screw_Terminal_01x03, J3 Screw_Terminal_01x03, J4 Screw_Terminal_01x02, J5 Screw_Terminal_01x03, J6 Screw_Terminal_01x03, J7 Screw_Terminal_01x02, J8 Conn_01x07_Female, P1 Digital, P10 CONN_01X01, P11 CONN_01X01, P12 CONN_01X01, P13 CONN_01X01, P2 Power, P3 Analog, P4 Analog, P5 PWM, P6 PWM, P7 Communication, P8 CONN_01X01, P9 CONN_01X01, U1 LM324A, U2 LM555xM, U3 LM555xM

Commit message: Add files via upload
Routing:
- net GND: track 80.6 -> 224.3 mm
- net IR_LADIES: track 125.0 -> 266.1 mm
- net INT2_REED_GENTS: track 182.6 -> 294.2 mm
